File: Origlia_Pablo/Ejercicio2/Ejercicio2.kicad_pcb (KiCad board)
At the start: 2 copper layers, 40.6 x 61 mm, 13 parts, among them J1 DB9-F, U1 AMIS42665TJAA1RG, U2 MAX232

Commit message: Agrego 3d. PO
Parts:
- added G***: LOGO, ej2:Logo_Poncho, F.Cu at (208.9, 111.1)
- added G101: Logo_OSHWA, ej2:Logo_OSHWA, F.Cu at (208.9, 62.9)
Routing:
- added copper zone on B.Cu, net GND
- added copper zone on F.Cu, net GND
Other:
- board text added: "INDUSTRIA ARGENTINA"
- board text added: "INTI - CMNB"
