File: Salguero_Federico/Ejercicio2/Salguero_Federico2.kicad_pcb (KiCad board)
At the start: 2 copper layers, 40.6 x 61 mm, 13 parts, among them J1 DB9, U1 AMIS42665TJAA1RG, U2 sp3232

Commit message: Version c/ modelos 3d
Parts:
- added G101: Logo_OSHWA, ej2:Logo_OSHWA, F.Cu at (136.8, 88.1)
- added Gxxx: LOGO, ej2:Logo_Poncho, F.Cu at (121.9, 134.1)
Routing:
- added copper zone on B.Cu, net GND
- added copper zone on F.Cu, net GND
Other:
- board text added: "Curso Kicad 12/2015 INTI - CMNB"
- board text added: "INDUSTRIA ARGENTINA"
