File: Salguero_Federico/Ejercicio2/Salguero_Federico2.kicad_pcb (KiCad board)
At the start: 2 copper layers, 40.6 x 61 mm, 15 parts, among them J1 DB9, U1 AMIS42665TJAA1RG, U2 sp3232

Commit message: Version final
Parts:
- moved G101 6.56 mm to (141.2, 93.0)
- moved R2 4.95 mm to (134.0, 121.0)
- moved R1 4.09 mm to (134.0, 126.7)
- moved C1 3.49 mm to (130.6, 127.6), turned to 0 degrees
- moved U1 2.42 mm to (134.5, 123.7), turned to 180 degrees
Connections:
- net Net-(JP1-Pad1) renamed /conector/CAN_P
- net Net-(JP1-Pad2) renamed /conector/CAN_N
Routing:
- net +5V: track 96.9 -> 113.9 mm
- net /conector/CAN_TX: track 23.3 -> 12.1 mm, vias 3 -> 1
- net /conector/CAN_RX: track 21.5 -> 10.3 mm
- net Net-(R1-Pad2): track 12.4 -> 18.4 mm
- net /conector/CAN_P: track 38.7 -> 33.2 mm
- net /conector/CAN_N: track 27.7 -> 29.4 mm
- net Net-(J1-Pad3): track 36.8 -> 35.5 mm
- net /conector/TXD: track 13.9 -> 12.8 mm
- net /conector/CTS: track 29.1 -> 28.1 mm
- net /conector/RXD: track 15.2 -> 14.6 mm
- removed copper zone on B.Cu, net GND
Other:
- net class Default: clearance 0.3048 -> 0.254
- rule trace_clearance: 0.3048 -> 0.254
- board text added: "1 oZ"
- board text added: "1,6"
- board text added: "FR4"
- board text added: "L1 Top"
- board text added: "L2 Top"
- board text added: "Terminacion: HASL E.Final: 1,6mm"
