File: Salguero_Federico/Ejercicio2/conector.sch (KiCad schematic (older format))
At the start: 6 parts, among them U1 AMIS42665TJAA1RG

Commit message: Version final
Connections:
- net CAN_N: now reaches JP1.2, R2.2, U1.6 (CANL)
- net CAN_P: now reaches JP1.1, R1.1, U1.7 (CANH)
Changed lines of the file:
@@
 Wire Wire Line
 	8600 3950 9250 3950
+Text Label 6250 3950 0    60   ~ 0
+CAN_P
+Text Label 6350 4150 0    60   ~ 0
+CAN_N
 $EndSCHEMATC
