File: Martina_Mauro/Ejercisio2/Ej2.kicad_pcb (KiCad board)
At the start: 2 copper layers, 40.6 x 61.1 mm, 13 parts, among them J1 DB9, U1 AMIS42665TJAA1RG, U2 RS232

Commit message: se sube modificacion en pcb
Parts:
- moved JP1 4.53 mm to (40.6, 115.2)
- moved U1 0.38 mm to (54.9, 116.5), turned to 180 degrees
- moved R1 0.28 mm to (55.2, 121.8)
- moved R2 0.28 mm to (55.2, 125.1)
Routing:
- net GND: track 0.00 -> 53.2 mm, vias 0 -> 13
- net /conector/CAN_RX: track 34.2 -> 19.6 mm
- net /conector/CAN_TX: track 26.6 -> 18.8 mm
- net /conector/CAN_N: track 32.3 -> 25.1 mm
- net Net-(R1-Pad2): track 6.82 -> 13.4 mm
- net /conector/CAN_P: track 22.8 -> 18.4 mm
- net +3.3V: track 26.7 -> 26.1 mm
- added copper zone on B.Cu, net GND
- added copper zone on F.Cu, net GND
Other:
- board text added: "FIUNER"
