File: Dmytrow_Ivan/Ejercicio2/Ejercicio2.kicad_pcb (KiCad board)
At the start: 2 copper layers, 40.6 x 61 mm, 13 parts, among them J1 DB9, U1 SSP3232, U2 AMIS42665TJAA1RG

Commit message: Subo los 3d shapes
Parts:
- turned C5 to 0 degrees
Routing:
- net +3.3V: track 21.8 -> 25.6 mm
- added copper zone on B.Cu, net GND
- added copper zone on F.Cu, net GND

Commit message: Subo el diseño con pares dif
Routing:
- net /Conector Ycan/CAN_P: track 23.1 -> 28.2 mm
- net /Conector Ycan/CAN_N: track 21.9 -> 26.3 mm
Other:
- board text added: "1Oz"
- board text added: "L1 Top [mixed]"
- board text added: "L2 Bot [mixed]"
- board text added: "Terminacion HASL"
- board text added: "dielectrico 1,6mm"
