File: Escobar_Martin/Ejercicio2/conector.sch (KiCad schematic (older format))
At the start: 6 parts, among them U1 AMIS42665TJAA1RG

Commit message: placa final
Connections:
- net CAN_N: now reaches JP1.2, R2.2, U1.6 (CANL)
- net CAN_P: now reaches JP1.3, R1.1, U1.7 (CANH)
Changed lines of the file:
@@
 Text HLabel 1700 2750 0    60   Input ~ 0
 RTS
+Text Label 6250 2050 0    60   ~ 0
+CAN_P
+Text Label 6250 2150 0    60   ~ 0
+CAN_N
 $EndSCHEMATC
