File: Escobar_Martin/Ejercicio2/Ejercicio2.kicad_pcb (KiCad board)
At the start: 2 copper layers, 40.6 x 61 mm, 13 parts, among them J1 DB9, U1 AMIS42665TJAA1RG, U2 ST232

Commit message: Ejercicio 2 n
Parts:
- added G***: LOGO, ej2:Logo_Poncho, F.Cu at (146.6, 131.3)

Commit message: con 3d
Parts:
- moved G*** 1.27 mm to (147.6, 130.6)
Routing:
- net GND: track 101.2 -> 104.5 mm, vias 0 -> 1
- added copper zone on B.Cu, net GND
- added copper zone on F.Cu, net GND
Other:
- board text added: "Industria Argentina"

Commit message: nuevo componente
Parts:
- moved R2 3.12 mm to (159.0, 145.8)
- moved R1 0.92 mm to (162.3, 141.2)
Routing:
- net Net-(JP1-Pad2): track 32.6 -> 29.3 mm
- net Net-(R1-Pad2): track 8.42 -> 5.99 mm
Changed lines of the file:
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@@
     (thickness 1.6)
     (drawings 5)
-    (tracks 205)
+    (tracks 204)
     (zones 0)
     (modules 14)
@@
   )
   (module ej2:R_1206_HandSoldering (layer F.Cu)
-    (at 161.544 141.732 270)
+    (at 162.306 141.224 270)
     (descr "Resistor SMD 1206, hand soldering")
     (tags "resistor 1206")
@@
   )
   (module ej2:R_1206_HandSoldering (layer F.Cu)
-    (at 157.353 148.463 180)
+    (at 158.972 145.796 180)
     (descr "Resistor SMD 1206, hand soldering")
     (tags "resistor 1206")
@@
     (pad 2 smd rect (at 1.8 0 270) (size 1.6 1.6) (layers F.Cu F.Paste)
       (net 2 +5V))
-    (model ${KIPRJMOD}/ej2.3dshapes/R_1206_HandSoldering.wrl
+    (model ${KIPRJMOD}/ej2.3dshapes/C_1206_HandSoldering.wrl
       (at (xyz 0 0 0))
       (scale (xyz 1 1 1))
@@
     (pad 2 smd rect (at 1.8 0 270) (size 1.6 1.6) (layers F.Cu F.Paste)
       (net 4 "Net-(C2-Pad2)"))
-    (model ${KIPRJMOD}/ej2.3dshapes/R_1206_HandSoldering.wrl
+    (model ${KIPRJMOD}/ej2.3dshapes/C_1206_HandSoldering.wrl
       (at (xyz 0 0 0))
       (scale (xyz 1 1 1))
@@
     (pad 2 smd rect (at 1.8 0) (size 1.6 1.6) (layers F.Cu F.Paste)
       (net 6 "Net-(C3-Pad2)"))
-    (model ${KIPRJMOD}/ej2.3dshapes/R_1206_HandSoldering.wrl
+    (model ${KIPRJMOD}/ej2.3dshapes/C_1206_HandSoldering.wrl
       (at (xyz 0 0 0))
       (scale (xyz 1 1 1))
@@
     (pad 2 smd rect (at 1.8 0) (size 1.6 1.6) (layers F.Cu F.Paste)
       (net 1 GND))
-    (model ${KIPRJMOD}/ej2.3dshapes/R_1206_HandSoldering.wrl
+    (model ${KIPRJMOD}/ej2.3dshapes/C_1206_HandSoldering.wrl
       (at (xyz 0 0 0))
       (scale (xyz 1 1 1))
@@
     (pad 2 smd rect (at 1.8 0) (size 1.6 1.6) (layers F.Cu F.Paste)
       (net 1 GND))
-    (model ${KIPRJMOD}/ej2.3dshapes/R_1206_HandSoldering.wrl
+    (model ${KIPRJMOD}/ej2.3dshapes/C_1206_HandSoldering.wrl
       (at (xyz 0 0 0))
       (scale (xyz 1 1 1))
@@
     (pad 2 smd rect (at 1.8 0) (size 1.6 1.6) (layers F.Cu F.Paste)
       (net 1 GND))
-    (model ${KIPRJMOD}/ej2.3dshapes/R_1206_HandSoldering.wrl
+    (model ${KIPRJMOD}/ej2.3dshapes/C_1206_HandSoldering.wrl
       (at (xyz 0 0 0))
       (scale (xyz 1 1 1))
@@
   (segment (start 144.526 126.238) (end 145.288 127) (width 0.3048) (layer F.Cu) (net 16))
   (segment (start 145.288 127) (end 155.38958 127) (width 0.3048) (layer F.Cu) (net 16))
+  (segment (start 156.972 142.748) (end 156.972 145.796) (width 0.3048) (layer F.Cu) (net 18))
   (segment (start 141.097 140.589) (end 142.621 140.589) (width 0.3048) (layer F.Cu) (net 18))
   (segment (start 157.099 142.113) (end 158.91 142.113) (width 0.3048) (layer F.Cu) (net 18))
@@
   (segment (start 147.574 135.636) (end 153.162 135.636) (width 0.3048) (layer F.Cu) (net 18))
   (segment (start 142.621 140.589) (end 147.574 135.636) (width 0.3048) (layer F.Cu) (net 18))
-  (segment (start 155.353 148.463) (end 155.353 146.653) (width 0.3048) (layer F.Cu) (net 18))
   (segment (start 157.607 142.113) (end 158.91 142.113) (width 0.3048) (layer F.Cu) (net 18))
   (segment (start 156.972 142.748) (end 157.607 142.113) (width 0.3048) (layer F.Cu) (net 18))
-  (segment (start 156.972 145.034) (end 156.972 142.748) (width 0.3048) (layer F.Cu) (net 18))
-  (segment (start 155.353 146.653) (end 156.972 145.034) (width 0.3048) (layer F.Cu) (net 18))
+  (segment (start 158.91 140.843) (end 160.401 140.843) (width 0.3048) (layer F.Cu) (net 19))
+  (segment (start 160.401 140.843) (end 161.512 139.732) (width 0.3048) (layer F.Cu) (net 19))
   (segment (start 141.097 138.049) (end 143.637 138.049) (width 0.3048) (layer F.Cu) (net 19))
   (segment (start 157.607 140.843) (end 158.91 140.843) (width 0.3048) (layer F.Cu) (net 19))
@@
   (segment (start 147.066 134.62) (end 153.67 134.62) (width 0.3048) (layer F.Cu) (net 19))
   (segment (start 143.637 138.049) (end 147.066 134.62) (width 0.3048) (layer F.Cu) (net 19))
-  (segment (start 158.91 140.843) (end 160.401 140.843) (width 0.3048) (layer F.Cu) (net 19))
-  (segment (start 160.401 140.843) (end 161.512 139.732) (width 0.3048) (layer F.Cu) (net 19))
   (segment (start 161.512 139.732) (end 161.544 139.732) (width 0.3048) (layer F.Cu) (net 19))
-  (segment (start 159.353 148.463) (end 159.353 145.923) (width 0.3048) (layer F.Cu) (net 20))
-  (segment (start 159.353 145.923) (end 161.544 143.732) (width 0.3048) (layer F.Cu) (net 20))
+  (segment (start 160.972 145.796) (end 161.122 145.796) (width 0.3048) (layer F.Cu) (net 20))
+  (segment (start 162.306 144.612) (end 162.306 143.224) (width 0.3048) (layer F.Cu) (net 20))
+  (segment (start 161.122 145.796) (end 162.306 144.612) (width 0.3048) (layer F.Cu) (net 20))
   (segment (start 158.91 143.383) (end 161.195 143.383) (width 0.3048) (layer F.Cu) (net 20))
   (segment (start 161.195 143.383) (end 161.544 143.732) (width 0.3048) (layer F.Cu) (net 20))
+  (segment (start 153.51 139.573) (end 154.305 139.573) (width 0.3048) (layer F.Cu) (net 21))
+  (segment (start 152.908 147.828) (end 152.908 149.86) (width 0.3048) (layer F.Cu) (net 21))
+  (segment (start 154.305 139.573) (end 155.194 140.462) (width 0.3048) (layer F.Cu) (net 21))
+  (segment (start 155.194 140.462) (end 155.194 145.542) (width 0.3048) (layer F.Cu) (net 21))
+  (segment (start 155.194 145.542) (end 152.908 147.828) (width 0.3048) (layer F.Cu) (net 21))
+  (segment (start 152.908 149.86) (end 153.924 150.876) (width 0.3048) (layer F.Cu) (net 21))
+  (segment (start 163.906201 137.490201) (end 162.382201 137.490201) (width 0.3048) (layer F.Cu) (net 21))
+  (segment (start 153.924 150.876) (end 163.068 150.876) (width 0.3048) (layer F.Cu) (net 21))
+  (segment (start 163.068 150.876) (end 164.084 149.86) (width 0.3048) (layer F.Cu) (net 21))
+  (segment (start 164.084 137.668) (end 163.906201 137.490201) (width 0.3048) (layer F.Cu) (net 21))
+  (segment (start 162.382201 137.490201) (end 161.544 136.652) (width 0.3048) (layer F.Cu) (net 21))
+  (segment (start 164.084 149.86) (end 164.084 137.668) (width 0.3048) (layer F.Cu) (net 21))
+  (segment (start 161.544 136.652) (end 161.544 135.382) (width 0.3048) (layer F.Cu) (net 21))
+  (segment (start 161.544 135.382) (end 162.306 134.62) (width 0.3048) (layer F.Cu) (net 21))
   (segment (start 170.18 134.62) (end 167.64 134.62) (width 0.3048) (layer F.Cu) (net 21))
-  (segment (start 154.305 139.573) (end 153.51 139.573) (width 0.3048) (layer F.Cu) (net 21))
-  (segment (start 155.194 140.462) (end 154.305 139.573) (width 0.3048) (layer F.Cu) (net 21))
-  (segment (start 155.194 145.542) (end 155.194 140.462) (width 0.3048) (layer F.Cu) (net 21))
-  (segment (start 152.908 147.828) (end 155.194 145.542) (width 0.3048) (layer F.Cu) (net 21))
-  (segment (start 152.908 149.86) (end 152.908 147.828) (width 0.3048) (layer F.Cu) (net 21))
-  (segment (start 153.924 150.876) (end 152.908 149.86) (width 0.3048) (layer F.Cu) (net 21))
-  (segment (start 163.068 150.876) (end 153.924 150.876) (width 0.3048) (layer F.Cu) (net 21))
-  (segment (start 164.084 149.86) (end 163.068 150.876) (width 0.3048) (layer F.Cu) (net 21))
-  (segment (start 164.084 138.176) (end 164.084 149.86) (width 0.3048) (layer F.Cu) (net 21))
-  (segment (start 163.576 137.668) (end 164.084 138.176) (width 0.3048) (layer F.Cu) (net 21))
-  (segment (start 162.052 137.668) (end 163.576 137.668) (width 0.3048) (layer F.Cu) (net 21))
-  (segment (start 161.544 137.16) (end 162.052 137.668) (width 0.3048) (layer F.Cu) (net 21))
-  (segment (start 161.544 135.382) (end 161.544 137.16) (width 0.3048) (layer F.Cu) (net 21))
-  (segment (start 162.306 134.62) (end 161.544 135.382) (width 0.3048) (layer F.Cu) (net 21))
   (via (at 162.306 134.62) (size 1.27) (drill 0.7112) (layers F.Cu B.Cu) (net 21))
   (segment (start 167.132 134.62) (end 162.306 134.62) (width 0.3048) (layer B.Cu) (net 21))
@@
     (connect_pads (clearance 0.508))
     (min_thickness 0.254)
-    (fill (arc_segments 32) (thermal_gap 0.508) (thermal_bridge_width 0.508))
+    (fill yes (arc_segments 32) (thermal_gap 0.508) (thermal_bridge_width 0.508))
     (polygon
       (pts
@@
     (connect_pads (clearance 0.508))
     (min_thickness 0.254)
-    (fill (arc_segments 32) (thermal_gap 0.508) (thermal_bridge_width 0.508))
+    (fill yes (arc_segments 32) (thermal_gap 0.508) (thermal_bridge_width 0.508))
     (polygon
       (pts
@@
     (min_thickness 0.254)
     (keepout (tracks allowed) (vias allowed) (copperpour not_allowed))
-    (fill (arc_segments 16) (thermal_gap 0.508) (thermal_bridge_width 0.508))
+    (fill yes (arc_segments 16) (thermal_gap 0.508) (thermal_bridge_width 0.508))
     (polygon
       (pts

Commit message: placa final
Connections:
- net Net-(JP1-Pad2) renamed /conector/CAN_N
- net Net-(JP1-Pad3) renamed /conector/CAN_P
Routing:
- net /conector/CAN_P: track 26.2 -> 46.9 mm
- net /conector/CAN_N: track 29.3 -> 45.0 mm
- net /conector/CAN_RX: track 46.4 -> 35.7 mm
- net /conector/CAN_TX: track 50.0 -> 39.3 mm
- net Net-(C5-Pad1): track 13.6 -> 13.0 mm
Other:
- board text added: "- - - - - -"
- board text added: "0,346 mm"
- board text added: "0,760 mm"
- board text added: "2 x 7628AT05 1 Oz"
- board text added: "4 x 7628M 1 Oz"
- board text added: "L1 Top (signal)"
- board text added: "L2 GND (Plate)"
- board text added: "L3 PWR (Mixed)"
- board text added: "L4 Bottom (Signal)"
- board text added: "Laminate Isola 1 Oz"
- board text added: "Prepeg Isola 1 Oz"
- board text added: "Stack - Up:"
- board text added: "Terminacion superficial: HASL Espesor final aproximado:1,6 mm"

Commit message: placa final
Routing:
- net GND: track 104.5 -> 131.2 mm, vias 1 -> 5
Other:
- net class Diff_90 added: clearance 1.778, trace_width 0.4572, via_dia 1.27, via_drill 0.7112
Changed lines of the file:
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@@
     (thickness 1.6)
     (drawings 25)
-    (tracks 376)
+    (tracks 394)
     (zones 0)
     (modules 14)
@@
     (add_net +3.3V)
     (add_net +5V)
-    (add_net /conector/CAN_N)
-    (add_net /conector/CAN_P)
     (add_net /conector/CAN_RX)
     (add_net /conector/CAN_TX)
@@
     (add_net "Net-(XA1-Pad8)")
     (add_net "Net-(XA1-Pad9)")
+  )
+  (net_class Diff_90 ""
+    (clearance 1.778)
+    (trace_width 0.4572)
+    (via_dia 1.27)
+    (via_drill 0.7112)
+    (uvia_dia 0.3)
+    (uvia_drill 0.1)
+    (add_net /conector/CAN_N)
+    (add_net /conector/CAN_P)
   )
   (module ej2:Logo_Poncho (layer TOP)
@@
   (gr_line (start 178.435 92.71) (end 137.795 92.71) (layer Edge.Cuts) (width 0.15))
   (gr_line (start 178.435 153.67) (end 178.435 92.71) (layer Edge.Cuts) (width 0.15))
+  (segment (start 172.72 147.32) (end 172.482 147.32) (width 0.3048) (layer TOP) (net 1))
+  (segment (start 172.482 147.32) (end 169.942 149.86) (width 0.3048) (layer TOP) (net 1))
+  (segment (start 169.942 149.86) (end 162.306 149.86) (width 0.3048) (layer TOP) (net 1))
+  (via (at 162.306 149.86) (size 1.27) (drill 0.7112) (layers TOP BOTTOM) (net 1))
+  (segment (start 158.75 133.604) (end 156.221111 133.604) (width 0.3048) (layer TOP) (net 1))
+  (segment (start 156.221111 133.604) (end 155.175591 131.940052) (width 0.3048) (layer TOP) (net 1))
+  (segment (start 155.175591 131.940052) (end 153.791539 130.556) (width 0.3048) (layer TOP) (net 1))
+  (segment (start 153.791539 130.556) (end 152.908 130.556) (width 0.3048) (layer TOP) (net 1))
+  (via (at 152.908 130.556) (size 1.27) (drill 0.7112) (layers TOP BOTTOM) (net 1))
+  (segment (start 160.169 131.191) (end 160.169 132.2958) (width 0.3048) (layer TOP) (net 1))
+  (segment (start 160.169 132.2958) (end 158.8608 133.604) (width 0.3048) (layer TOP) (net 1))
+  (segment (start 158.8608 133.604) (end 158.75 133.604) (width 0.3048) (layer TOP) (net 1))
+  (via (at 158.75 133.604) (size 1.27) (drill 0.7112) (layers TOP BOTTOM) (net 1))
+  (segment (start 142.6718 142.748) (end 144.018 142.748) (width 0.3048) (layer TOP) (net 1))
+  (segment (start 144.018 142.748) (end 145.288 141.478) (width 0.3048) (layer TOP) (net 1))
+  (via (at 145.288 141.478) (size 1.27) (drill 0.7112) (layers TOP BOTTOM) (net 1))
+  (segment (start 141.097 143.129) (end 142.2908 143.129) (width 0.3048) (layer TOP) (net 1))
+  (segment (start 142.2908 143.129) (end 142.6718 142.748) (width 0.3048) (layer TOP) (net 1))
   (segment (start 162.306 112.014) (end 162.306 113.284) (width 0.3048) (layer BOTTOM) (net 1))
   (segment (start 160.445 113.03) (end 162.052 113.03) (width 0.3048) (layer TOP) (net 1))
