File: Mainenti_Miguel/Ejercicio2/conector.sch (KiCad schematic (older format))
At the start: 6 parts, among them U1 AMIS42665TJAA1RG

Commit message: ruteo del par diferencial y ecualizado
Connections:
- net labels added: CAN_N, CAN_P
Changed lines of the file:
@@
 Text Label 8800 3000 0    60   ~ 0
 CAN_TX
+Text Label 6100 2900 0    60   ~ 0
+CAN_P
+Text Label 6100 3000 0    60   ~ 0
+CAN_N
 $EndSCHEMATC
