File: Sisevich_Pablo/Ejercicio_2/Ejercicio_2.kicad_pcb (KiCad board)
At the start: 2 copper layers, 13 parts, among them J1 DB9, U1 AMIS42665TJAA1RG, U2 SP-232v2

Commit message: Actualizo PCB
Routing:
- net GND: track 21.9 -> 43.4 mm, vias 6 -> 18
- added copper zone on B.Cu, net GND
- added copper zone on F.Cu, net GND
Other:
- board text added: "IND.ARG."
- board text added: "INTI-CNMB"
Changed lines of the file:
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@@
   (general
     (links 44)
-    (no_connects 17)
-    (area 0 0 0 0)
+    (no_connects 0)
+    (area 101.276499 63.838499 148.055001 125.195001)
     (thickness 1.6)
-    (drawings 5)
-    (tracks 174)
+    (drawings 7)
+    (tracks 201)
     (zones 0)
     (modules 13)
@@
     (user_trace_width 0.3048)
     (trace_clearance 0.2)
-    (zone_clearance 0.508)
-    (zone_45_only no)
+    (zone_clearance 0.2032)
+    (zone_45_only yes)
     (trace_min 0.2)
     (segment_width 0.2)
@@
     )
   )
+  (gr_text INTI-CNMB (at 117.348 123.063) (layer F.Cu)
+    (effects (font (size 1.5 1.5) (thickness 0.3)))
+  )
   (gr_line (start 107.315 64.135) (end 107.315 125.095) (angle 90) (layer Eco2.User) (width 0.2))
+  (gr_text "IND.ARG.\n" (at 116.586 122.936) (layer B.Cu)
+    (effects (font (size 1.5 1.5) (thickness 0.3)) (justify mirror))
+  )
   (gr_line (start 147.955 64.135) (end 107.315 64.135) (angle 90) (layer Eco2.User) (width 0.2))
   (gr_line (start 147.955 95.25) (end 147.955 64.135) (angle 90) (layer Eco2.User) (width 0.2))
   (gr_line (start 147.955 125.095) (end 147.955 95.25) (angle 90) (layer Eco2.User) (width 0.2))
   (gr_line (start 107.315 125.095) (end 147.955 125.095) (angle 90) (layer Eco2.User) (width 0.2))
+  (segment (start 123.952 72.644) (end 125.095 72.644) (width 0.3048) (layer F.Cu) (net 1))
+  (via (at 125.095 74.549) (size 1.27) (drill 0.7112) (layers F.Cu B.Cu) (net 1))
+  (segment (start 127 74.549) (end 125.095 74.549) (width 0.3048) (layer B.Cu) (net 1))
+  (via (at 127 74.549) (size 1.27) (drill 0.7112) (layers F.Cu B.Cu) (net 1))
+  (segment (start 127 72.644) (end 127 74.549) (width 0.3048) (layer F.Cu) (net 1))
+  (via (at 127 72.644) (size 1.27) (drill 0.7112) (layers F.Cu B.Cu) (net 1))
+  (segment (start 125.095 72.644) (end 127 72.644) (width 0.3048) (layer B.Cu) (net 1))
+  (via (at 125.095 72.644) (size 1.27) (drill 0.7112) (layers F.Cu B.Cu) (net 1))
+  (segment (start 115.951 112.522) (end 117.348 112.522) (width 0.3048) (layer F.Cu) (net 1))
+  (via (at 117.348 114.3) (size 1.27) (drill 0.7112) (layers F.Cu B.Cu) (net 1))
+  (segment (start 119.126 114.3) (end 117.348 114.3) (width 0.3048) (layer B.Cu) (net 1))
+  (via (at 119.126 114.3) (size 1.27) (drill 0.7112) (layers F.Cu B.Cu) (net 1))
+  (segment (start 119.126 112.649) (end 119.126 114.3) (width 0.3048) (layer F.Cu) (net 1))
+  (segment (start 119.253 112.522) (end 119.126 112.649) (width 0.3048) (layer F.Cu) (net 1))
+  (via (at 119.253 112.522) (size 1.27) (drill 0.7112) (layers F.Cu B.Cu) (net 1))
+  (segment (start 117.348 112.522) (end 119.253 112.522) (width 0.3048) (layer B.Cu) (net 1))
+  (via (at 117.348 112.522) (size 1.27) (drill 0.7112) (layers F.Cu B.Cu) (net 1))
+  (segment (start 114.554 99.314) (end 115.57 99.314) (width 0.3048) (layer F.Cu) (net 1))
+  (via (at 121.031 99.314) (size 1.27) (drill 0.7112) (layers F.Cu B.Cu) (net 1))
+  (segment (start 119.126 99.314) (end 121.031 99.314) (width 0.3048) (layer B.Cu) (net 1))
+  (via (at 119.126 99.314) (size 1.27) (drill 0.7112) (layers F.Cu B.Cu) (net 1))
+  (segment (start 117.348 99.314) (end 119.126 99.314) (width 0.3048) (layer F.Cu) (net 1))
+  (via (at 117.348 99.314) (size 1.27) (drill 0.7112) (layers F.Cu B.Cu) (net 1))
+  (segment (start 117.221 99.314) (end 117.348 99.314) (width 0.3048) (layer B.Cu) (net 1))
+  (segment (start 117.856 99.314) (end 117.221 99.314) (width 0.3048) (layer B.Cu) (net 1))
+  (segment (start 115.57 99.314) (end 117.856 99.314) (width 0.3048) (layer B.Cu) (net 1))
+  (via (at 115.57 99.314) (size 1.27) (drill 0.7112) (layers F.Cu B.Cu) (net 1))
   (segment (start 132.969 89.281) (end 133.731 89.281) (width 0.3048) (layer F.Cu) (net 1))
   (via (at 133.858 89.408) (size 1.27) (drill 0.7112) (layers F.Cu B.Cu) (net 1))
@@
   (segment (start 124.333 82.296) (end 124.079 82.042) (width 0.3048) (layer F.Cu) (net 1))
   (segment (start 130.86842 89.281) (end 132.969 89.281) (width 0.3048) (layer F.Cu) (net 1))
-  (segment (start 132.969 89.281) (end 133.731 89.281) (width 0.3048) (layer F.Cu) (net 1) (status 2))
+  (segment (start 132.969 89.281) (end 133.731 89.281) (width 0.3048) (layer F.Cu) (net 1))
   (segment (start 121.285 82.455) (end 121.285 84.074) (width 0.3048) (layer F.Cu) (net 2))
   (segment (start 122.301 84.455) (end 122.809 84.963) (width 0.3048) (layer F.Cu) (net 2))
@@
   (segment (start 118.2624 82.2706) (end 119.7356 82.2706) (width 0.3048) (layer B.Cu) (net 9))
   (via (at 128.27 90.551) (size 1.27) (drill 0.7112) (layers F.Cu B.Cu) (net 9))
-  (segment (start 128.27 90.551) (end 130.86842 90.551) (width 0.3048) (layer F.Cu) (net 9) (status 800000))
+  (segment (start 128.27 90.551) (end 130.86842 90.551) (width 0.3048) (layer F.Cu) (net 9))
   (segment (start 121.031 90.551) (end 128.27 90.551) (width 0.3048) (layer B.Cu) (net 9))
   (segment (start 120.396 89.916) (end 121.031 90.551) (width 0.3048) (layer B.Cu) (net 9))
@@
   (segment (start 118.2624 79.502) (end 121.031 79.502) (width 0.3048) (layer B.Cu) (net 10))
   (segment (start 128.524 91.821) (end 128.27 92.202) (width 0.3048) (layer F.Cu) (net 10))
-  (segment (start 128.524 91.821) (end 130.86842 91.821) (width 0.3048) (layer F.Cu) (net 10) (status 800000))
+  (segment (start 128.524 91.821) (end 130.86842 91.821) (width 0.3048) (layer F.Cu) (net 10))
   (via (at 128.27 92.202) (size 1.27) (drill 0.7112) (layers F.Cu B.Cu) (net 10))
   (segment (start 129.54 89.916) (end 129.54 90.424) (width 0.3048) (layer B.Cu) (net 10))
@@
   (segment (start 135.636 94.996) (end 135.636 97.536) (width 0.3048) (layer F.Cu) (net 21))
   (segment (start 135.001 94.361) (end 135.636 94.996) (width 0.3048) (layer F.Cu) (net 21))
-  (segment (start 130.778 110.617) (end 128.778 110.617) (width 0.3048) (layer F.Cu) (net 22) (status 400000))
+  (segment (start 130.778 110.617) (end 128.778 110.617) (width 0.3048) (layer F.Cu) (net 22))
   (segment (start 145.415 120.523) (end 145.415 71.12) (width 0.3048) (layer F.Cu) (net 22))
   (segment (start 129.413 104.775) (end 128.778 105.41) (width 0.3048) (layer F.Cu) (net 22))
@@
   (segment (start 129.54 121.158) (end 144.78 121.158) (width 0.3048) (layer F.Cu) (net 22))
   (segment (start 144.78 121.158) (end 145.415 120.523) (width 0.3048) (layer F.Cu) (net 22))
-  (segment (start 131.224 104.775) (end 129.413 104.775) (width 0.3048) (layer F.Cu) (net 22) (status 400000))
-  (segment (start 144.78 70.485) (end 142.24 70.485) (width 0.3048) (layer F.Cu) (net 22) (status 800000))
+  (segment (start 131.224 104.775) (end 129.413 104.775) (width 0.3048) (layer F.Cu) (net 22))
+  (segment (start 144.78 70.485) (end 142.24 70.485) (width 0.3048) (layer F.Cu) (net 22))
   (segment (start 145.415 71.12) (end 144.78 70.485) (width 0.3048) (layer F.Cu) (net 22))
+  (zone (net 1) (net_name GND) (layer F.Cu) (hatch edge 0.508)
+    (connect_pads (clearance 0.2032))
+    (min_thickness 0.2032)
+    (fill yes (arc_segments 32) (thermal_gap 0.2032) (thermal_bridge_width 0.508))
+    (polygon
+      (pts
+        (xy 147.955 64.135) (xy 147.955 125.095) (xy 127.762 125.095) (xy 127.762 121.031) (xy 107.315 121.031)
+        (xy 107.315 64.135) (xy 147.955 64.135)
+      )
+    )
+  )
+  (zone (net 1) (net_name GND) (layer B.Cu) (hatch edge 0.508)
+    (connect_pads (clearance 0.2032))
+    (min_thickness 0.2032)
+    (fill yes (arc_segments 32) (thermal_gap 0.2032) (thermal_bridge_width 0.508))
+    (polygon
+      (pts
+        (xy 147.955 125.095) (xy 127.762 125.095) (xy 127.762 121.031) (xy 107.315 121.031) (xy 107.315 64.135)
+        (xy 147.955 64.135) (xy 147.955 125.095)
+      )
+    )
+  )
+  (zone (net 0) (net_name "") (layer F.Cu) (hatch edge 0.508)
+    (connect_pads (clearance 0.2032))
+    (min_thickness 0.2032)
+    (keepout (tracks not_allowed) (vias not_allowed) (copperpour not_allowed))
+    (fill (arc_segments 32) (thermal_gap 0.2032) (thermal_bridge_width 0.508))
+    (polygon
+      (pts
+        (xy 124.206 102.235) (xy 126.873 102.235) (xy 126.873 108.077) (xy 124.206 108.077) (xy 121.666 110.617)
+        (xy 114.427 110.617) (xy 112.141 108.331) (xy 109.093 108.331) (xy 109.093 102.743) (xy 112.141 102.743)
+        (xy 114.681 100.203) (xy 122.174 100.203) (xy 124.206 102.235)
+      )
+    )
+  )
 )

Commit message: Actualizo PCB
Routing:
- net GND: track 43.4 -> 21.9 mm, vias 18 -> 6
- net (no net): track 0.00 -> 21.5 mm, vias 0 -> 12

Commit message: Actualizo PCB
Parts:
- added G***: LOGO, ej2:Logo_Poncho, F.Cu at (128.7, 116.6)
- added G101: Logo_OSHWA, ej2:Logo_OSHWA, F.Cu at (125.7, 67.8)
Connections:
- net Net-(JP1-Pad1) renamed /Conector y Can/CAN_P
- net Net-(JP1-Pad2) renamed /Conector y Can/CAN_N
Routing:
- net /Conector y Can/CAN_P: track 18.3 -> 30.8 mm
- net /Conector y Can/CAN_N: track 18.5 -> 30.9 mm
- net (no net): track 21.5 -> 18.0 mm
Other:
- board text added: "1 Oz"
- board text added: "Dielectrico"
- board text added: "Espesor final aprox: 1,6mm"
- board text added: "L1 Top (Mixed)"
- board text added: "L2 Bottom (Mixed)"
- board text added: "Stack-UP"
- board text added: "Terminación superficial: HASL"
