File: Sisevich_Pablo/Ejercicio_2/conector.sch (KiCad schematic (older format))
At the start: 6 parts, among them U1 AMIS42665TJAA1RG

Commit message: Actualizo PCB
Connections:
- net CAN_N: now also JP1.2, R2.2, U1.6 (CANL)
- net CAN_P: now also JP1.1, R1.1, U1.7 (CANH)
Changed lines of the file:
@@
 Wire Wire Line
 	9400 3350 9400 4100
-Text Label 6750 3400 0    60   ~ 0
+Text Label 6850 3400 0    60   ~ 0
 CAN_P
-Text Label 6750 3500 0    60   ~ 0
+Text Label 6900 3500 0    60   ~ 0
 CAN_N
 NoConn ~ 3650 4350
