File: Fusari_Diego/Ejercicio2/Conector.sch (KiCad schematic (older format))
At the start: 6 parts, among them U1 AMIS42665TJAA1RG

Commit message: Al pcb se le agregaron los controles de impedancias
Connections:
- net CAN_N: now reaches CAN1.2, R2.2, U1.6 (CANL)
- net CAN_P: now reaches CAN1.3, R1.1, U1.7 (CANH)
Changed lines of the file:
@@
 Wire Wire Line
 	3700 5250 2750 5250
+Text Label 6900 4400 0    60   ~ 0
+CAN_P
+Text Label 6900 4500 0    60   ~ 0
+CAN_N
 $EndSCHEMATC
