File: Laiuppa_Adrian/Ejercicio_2/ej2.kicad_pcb (KiCad board)
At the start: 2 copper layers, 40.6 x 61 mm, 15 parts, among them J1 DB9, U1 AMIS42665TJAA1RG, U2 SP3232V2

Commit message: plano de tierra y 3d
Parts:
- moved C6 7.32 mm to (74.5, 93.9)
Routing:
- net GND: track 21.8 -> 11.7 mm, vias 8 -> 4
- net +5V: track 79.6 -> 71.2 mm, vias 0 -> 1
- net (no net): track 0.00 -> 4.99 mm, vias 0 -> 4
- added copper zone on B.Cu, net GND
- added copper zone on F.Cu, net GND

Commit message: Signed-off-by: Laiuppa Adrian <alaiuppa@gmail.com>
par diferencial
Routing:
- net /conector y can/CAN_N: track 32.1 -> 39.4 mm, vias 1 -> 2
- net /conector y can/CAN_P: track 37.2 -> 31.5 mm, vias 0 -> 1
Other:
- board text added: "Stack - UP: 1 Oz ______ ______ ______ ______ L1 Top (Mixer) DIELECTRICO 1,6mm 1 Oz ______ ______ ______ ______ L1 Bot (Mixer) Terminacion superficial: HASL Espesor final aproximado: 1,6mm"
