File: Cuenca_Gonzalo/ejercicio_2/Ej2.kicad_pcb (KiCad board)
At the start: 2 copper layers, 40.6 x 61 mm, 13 parts, among them J1 DB9, J2 CAN, U1 SP3232_V2, U2 AMIS42665TJAA1RG

Commit message: GoCu Agregado los planos y la vista 3D
Parts:
- added G***: LOGO, ej2:Logo_Poncho, F.Cu at (87.4, 100.3)
- added G101: Logo_OSHWA, ej2:Logo_OSHWA, F.Cu at (77.5, 100.6)
Routing:
- net GND: track 0.00 -> 24.8 mm, vias 0 -> 4
- net /Conector y Can/CAN_P: track 22.6 -> 23.6 mm
- added copper zone on B.Cu, net GND
- added copper zone on F.Cu, net GND
Other:
- board text added: "Curso KiCad INTI"
- board text added: "Gonzalo Cuenca"

Commit message: Agrego el ruteo del CAN
Parts:
- renumbered C2 to C1, C3 to C1, C4 to C1, C5 to C1, C6 to C1, G*** to G***1, J2 to J1, R2 to R1, U2 to U1
Routing:
- net /Conector y Can/CAN_N: track 28.6 -> 25.2 mm
- net +5V: track 47.7 -> 49.2 mm
- net /Conector y Can/CAN_P: track 23.6 -> 22.2 mm
- net (no net): track 0.00 -> 1.27 mm, vias 0 -> 1
Other:
- board text added: "1 Oz"
- board text added: "1,6mm"
- board text added: "Dieléctrico"
- board text added: "L1 Top(Mixed) L2 Bottom(Mixed)"
- board text added: "Stack -UP:"
- board text added: "Terminación superficial: HASL Espesor final aproximado: 1,6mm"
